File: concierge-door-node.sch (KiCad schematic (older format))
At the start: 3 parts, among them U1 NodeMCU_Amica_R2

Commit message: Cryptochip and Stepstick added to project.
Parts:
- added U2: ATECC508A, Housings_SOIC:SOIC-8-1EP_3.9x4.9mm_Pitch1.27mm, symbol ATECC508A
- added U3: POLOLU_A4988, symbol POLOLU_A4988
- gave numbers to parts that had none: 2
Changed lines of the file:
@@
 LIBS:rfid-rc522-module
 LIBS:nodemcu
+LIBS:atecc508a
+LIBS:pololu_a4988
 LIBS:concierge-door-node-cache
 EELAYER 25 0
@@
 F 0 "U1" H 4250 3150 50  0000 C CNN
 F 1 "NodeMCU_Amica_R2" H 4250 1500 50  0000 C CNN
-F 2 "" H 4500 2350 50  0000 C CNN
+F 2 "" H 4500 2350 50  0001 C CNN
 F 3 "" H 4500 2350 50  0000 C CNN
 	1    4250 2350
@@
 	3400 1600 4000 1600
 $Comp
-L GND #PWR04
+L GND #PWR3
 U 1 1 572E4B65
 P 3600 3100
-F 0 "#PWR04" H 3600 2850 50  0001 C CNN
+F 0 "#PWR3" H 3600 2850 50  0001 C CNN
 F 1 "GND" H 3600 2950 50  0000 C CNN
 F 2 "" H 3600 3100 50  0000 C CNN
@@
 $EndComp
 $Comp
-L +3.3V #PWR05
+L +3.3V #PWR1
 U 1 1 572E4BF4
 P 3150 2850
-F 0 "#PWR05" H 3150 2700 50  0001 C CNN
+F 0 "#PWR1" H 3150 2700 50  0001 C CNN
 F 1 "+3.3V" H 3150 2990 50  0000 C CNN
 F 2 "" H 3150 2850 50  0000 C CNN
@@
 NoConn ~ 4950 2800
 $Comp
-L PWR_FLAG #FLG07
+L PWR_FLAG #FLG2
 U 1 1 572E8587
 P 4000 1550
-F 0 "#FLG07" H 4000 1645 50  0001 C CNN
+F 0 "#FLG2" H 4000 1645 50  0001 C CNN
 F 1 "PWR_FLAG" H 4000 1730 50  0000 C CNN
 F 2 "" H 4000 1550 50  0000 C CNN
@@
 Connection ~ 3550 1600
 $Comp
-L PWR_FLAG #FLG08
+L PWR_FLAG #FLG1
 U 1 1 572E8681
 P 2850 2850
-F 0 "#FLG08" H 2850 2945 50  0001 C CNN
+F 0 "#FLG1" H 2850 2945 50  0001 C CNN
 F 1 "PWR_FLAG" H 2850 3030 50  0000 C CNN
 F 2 "" H 2850 2850 50  0000 C CNN
@@
 Connection ~ 3150 2950
 $Comp
-L GND #PWR010
+L GND #PWR6
 U 1 1 572F7C0D
 P 4350 3200
-F 0 "#PWR010" H 4350 2950 50  0001 C CNN
+F 0 "#PWR6" H 4350 2950 50  0001 C CNN
 F 1 "GND" H 4350 3050 50  0000 C CNN
 F 2 "" H 4350 3200 50  0000 C CNN
@@
 	4350 2800 4350 3200
 $Comp
-L +3.3V #PWR012
+L +3.3V #PWR5
 U 1 1 572F7C98
 P 4200 1650
-F 0 "#PWR012" H 4200 1500 50  0001 C CNN
+F 0 "#PWR5" H 4200 1500 50  0001 C CNN
 F 1 "+3.3V" H 4200 1790 50  0000 C CNN
 F 2 "" H 4200 1650 50  0000 C CNN
@@
 	3950 1650 3950 1900
 $Comp
-L GND #PWR013
+L GND #PWR4
 U 1 1 572F7CDF
 P 3800 1700
-F 0 "#PWR013" H 3800 1450 50  0001 C CNN
+F 0 "#PWR4" H 3800 1450 50  0001 C CNN
 F 1 "GND" H 3800 1550 50  0000 C CNN
 F 2 "" H 3800 1700 50  0000 C CNN
@@
 NoConn ~ 4850 2450
 $Comp
-L SPST SW?
+L SPST SW1
 U 1 1 575B1D56
 P 3500 4100
-F 0 "SW?" H 3500 4200 50  0000 C CNN
+F 0 "SW1" H 3500 4200 50  0000 C CNN
 F 1 "SPST" H 3500 4000 50  0000 C CNN
-F 2 "" H 3500 4100 50  0000 C CNN
+F 2 "" H 3500 4100 50  0001 C CNN
 F 3 "" H 3500 4100 50  0000 C CNN
 	1    3500 4100
@@
 $EndComp
 $Comp
-L SPST SW?
+L SPST SW2
 U 1 1 575B1DBB
 P 3500 4500
-F 0 "SW?" H 3500 4600 50  0000 C CNN
+F 0 "SW2" H 3500 4600 50  0000 C CNN
 F 1 "SPST" H 3500 4400 50  0000 C CNN
-F 2 "" H 3500 4500 50  0000 C CNN
+F 2 "" H 3500 4500 50  0001 C CNN
 F 3 "" H 3500 4500 50  0000 C CNN
 	1    3500 4500
@@
 $EndComp
 $Comp
-L +12V #PWR?
+L +12V #PWR2
 U 1 1 5956132C
 P 3400 1550
-F 0 "#PWR?" H 3400 1400 50  0001 C CNN
+F 0 "#PWR2" H 3400 1400 50  0001 C CNN
 F 1 "+12V" H 3400 1690 50  0000 C CNN
 F 2 "" H 3400 1550 50  0001 C CNN
@@
 Wire Wire Line
 	3400 1600 3400 1550
+$Comp
+L ATECC508A U2
+U 1 1 59669691
+P 8050 2400
+F 0 "U2" H 7650 2750 50  0000 L CNN
+F 1 "ATECC508A" H 8150 2750 50  0000 L CNN
+F 2 "Housings_SOIC:SOIC-8-1EP_3.9x4.9mm_Pitch1.27mm" H 8050 1850 50  0001 C CNN
+F 3 "" H 8050 1850 50  0000 C CNN
+	1    8050 2400
+	1    0    0    -1
+$EndComp
+$Comp
+L POLOLU_A4988 U3
+U 1 1 5966985A
+P 6800 3600
+F 0 "U3" H 6800 4050 60  0000 C CNN
+F 1 "POLOLU_A4988" V 6800 3600 50  0000 C CNN
+F 2 "" H 6800 3600 60  0001 C CNN
+F 3 "" H 6800 3600 60  0000 C CNN
+	1    6800 3600
+	1    0    0    -1
+$EndComp
 $EndSCHEMATC
